File: KiCad/Z80-FDC-V2.kicad_pcb (KiCad board)
At the start: 2 copper layers, 101.6 x 53.3 mm, 35 parts, among them J1 Floppy, J2 Floppy 5V, J3 RCBus-80, U1 37C65, U2 DS1302+, U3 ATF16V8B, U4 74HCT174, U5 74HCT125, U6 74LVC1G06, Y1 16MHz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

Commit message: Update KiCad and add Gerber for V2.0
Signed-off-by: Sergey Kiselev <skiselev@gmail.com>
Parts:
- removed U6: 74LVC1G06, Package_TO_SOT_SMD:SOT-23-5_HandSoldering
- added J4: GPIO, My_Components:Conn_Pin_Header_5x1_2.54mm, F.Cu at (224.8, 111.8)
- JP2: value INT_Select -> RTC_ENA; footprint My_Components:Conn_Pin_Header_4x2_2.54mm -> Jumper:SolderJumper-3_P1.3mm_Bridged12_RoundedPad1.0x1.5mm_NumberLabels; moved to B.Cu
- JP3: footprint My_Components:Conn_Pin_Header_3x1_2.54mm -> Jumper:SolderJumper-3_P1.3mm_Bridged12_RoundedPad1.0x1.5mm_NumberLabels; moved to B.Cu
- R1, R2, R3: value 4.7k -> 10k
- U4: value 74HCT174 -> 74AHCT174
- moved JP2 57.1 mm to (167.6, 94.6), turned to 180 degrees
- moved C9 7.73 mm to (222.2, 94.0), turned to 0 degrees
- moved C10 6.55 mm to (219.7, 105.7), turned to 90 degrees
- moved C8 6.35 mm to (222.2, 99.1)
- moved C11 5.24 mm to (219.7, 113.0), turned to -90 degrees
- moved Y3 4.58 mm to (214.6, 109.2), turned to 90 degrees
- moved JP3 4.02 mm to (214.6, 102.9), turned to 180 degrees
- moved Y1 3.81 mm to (214.6, 96.5), turned to -90 degrees
- moved LOGO1 3.17 mm to (196.8, 118.1)
- moved LOGO2 3.17 mm to (196.8, 119.4)
- renumbered LOGO1 to LOGO2, LOGO2 to LOGO3
Connections:
- J3 pad 22: /~{INT} -> unconnected-(J3-Pad22)
- J3 pad 37: /~{IRQ1} -> unconnected-(J3-Pad37)
- J3 pad 66: /~{NMI} -> unconnected-(J3-Pad66)
- J3 pad 77: /~{IRQ2} -> unconnected-(J3-Pad77)
- JP2 pad 1: /~{INT} -> /~{RTC_RD}
- JP2 pad 2: /~{IRQ_OD} -> /~{RTC_RD_ENA}
- JP2 pad 3: /~{NMI} -> VCC
- R3 pad 1: GND -> VCC
- R3 pad 2: /~{IRQ} -> /IN_D7
- U2 pad 7: /RTC_CLK -> /RTC_SCLK
- U4 pad 10: unconnected-(U4-Pad10) -> /OUT_D0
- U4 pad 12: unconnected-(U4-Pad12) -> /RTC_DOUT
- U4 pad 13: /D3 -> /D7
- U4 pad 14: /D5 -> /D4
- U4 pad 15: /RTC_WE -> /RTC_CE
- U4 pad 2: /RTC_CE -> /~{RTC_WE}
- U4 pad 3: /D4 -> /D5
- U4 pad 4: /D7 -> /D6
- U4 pad 5: /RTC_IN -> /RTC_SCLK
- U4 pad 6: /D6 -> /D2
- U4 pad 7: /RTC_CLK -> /OUT_D2
- U5 pad 10: /~{RTC_RD} -> /~{RTC_RD_ENA}
- U5 pad 12: /RTC_IN -> /RTC_DOUT
- U5 pad 13: /RTC_WE -> /~{RTC_WE}
- U5 pad 4: /IRQ -> /~{RTC_RD_ENA}
- U5 pad 5: VCC -> /IN_D7
- U5 pad 6: /~{IRQ} -> /D7
- Y2 pad 3: (no net) -> GND
Routing:
- net GND: track 676.3 -> 559.6 mm, vias 11 -> 12
- net /IN_D7: track 0.00 -> 78.8 mm, vias 0 -> 1
- net /~{IRQ}: track 73.6 -> 0.00 mm, vias 1 -> 0
- net /RTC_CLK: track 67.3 -> 0.00 mm, vias 1 -> 0
- net /RTC_SCLK: track 0.00 -> 67.3 mm, vias 0 -> 1
- net /OUT_D0: track 0.00 -> 59.4 mm, vias 0 -> 1
- net /IRQ: track 58.1 -> 0.00 mm, vias 1 -> 0
- net /OUT_D2: track 0.00 -> 57.6 mm
- net /D2: track 16.3 -> 70.6 mm
- net /~{INT}: track 40.2 -> 0.00 mm
- net /RTC_IN: track 32.6 -> 0.00 mm
- net /D3: track 51.6 -> 19.9 mm
- net /~{RTC_WE}: track 0.00 -> 31.5 mm
- net /~{NMI}: track 30.0 -> 0.00 mm
- net /RTC_DOUT: track 0.00 -> 28.6 mm
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Other:
- board text added: "+5V"
- board text added: "Design files and documentation: Licensed under CERN-OHL-S:"
- board text added: "GND"
- board text added: "IN_D7"
- board text added: "Jumpers settings [default]: JP2: [1-2]: Enable RTC JP2: 2-3 : Disable RTC JP3: [1-2]: Y3 crystal not installed disable 300 Kbps transfer rate JP3: 2-3 : Y3 crystal installed enable 300 Kbps transfer rate"
- board text added: "OUT_D0"
- board text added: "OUT_D2"
- board text added: "SK102"
- board text added: "Y3, C10, and C11 are optional; required for 300 Kbps transfer rate support"
- board text added: "https://github.com/skiselev/flock-v2 https://cern-ohl.web.cern.ch"
- board text removed: "Design files and documentation: github.com/skiselev/flock-v2"
- board text removed: "Jumpers settings: JP2: Open: Disable interrupts JP3: Installed: Select interrupt pin JP3: 1-2: Y3 crystal not installed disable 300 Kbps transfer rate JP3: 2-3: Y3 crystal installed enable 300 Kbps transfer rate"
- board text removed: "Licensed under CERN-OHL-S: https://cern-ohl.web.cern.ch"
- board text removed: "~{INT}"
- board text removed: "~{IRQ0}"
- board text removed: "~{IRQ1}"
- board text removed: "~{NMI}"
