File: KiCad/Z80-FDC-V2.kicad_sch (KiCad schematic)
At the start: 35 parts, among them J1 Floppy, J2 Floppy 5V, J3 RCBus-80, U1 37C65, U2 DS1302+, U3 ATF16V8B, U4 74HCT174, U5 74HCT125, U6 74LVC1G06, Y1 16MHz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

Commit message: Update KiCad and add Gerber for V2.0
Signed-off-by: Sergey Kiselev <skiselev@gmail.com>
Parts:
- removed JP2: INT_Select, My_Components:Conn_Pin_Header_4x2_2.54mm, symbol Connector_Generic:Conn_02x04_Odd_Even
- removed U6: 74LVC1G06, Package_TO_SOT_SMD:SOT-23-5_HandSoldering, symbol 74xGxx:74LVC1G06
- added J4: GPIO, My_Components:Conn_Pin_Header_5x1_2.54mm, symbol Connector_Generic:Conn_01x05
- added JP2: RTC_ENA, Jumper:SolderJumper-3_P1.3mm_Bridged12_RoundedPad1.0x1.5mm_NumberLabels, symbol Jumper:Jumper_3_Bridged12
- JP3: footprint My_Components:Conn_Pin_Header_3x1_2.54mm -> Jumper:SolderJumper-3_P1.3mm_Bridged12_RoundedPad1.0x1.5mm_NumberLabels
- R1, R2, R3: value 4.7k -> 10k
- U4: value 74HCT174 -> 74AHCT174
- Y2: symbol Device:Crystal_Small -> Device:Crystal_GND3_Small
Connections:
- net D2: now also U4.6 (D2)
- net D3: no longer U4.13 (D4)
- net D4: now also U4.14 (D5); no longer U4.3 (D0)
- net D5: now also U4.3 (D0); no longer U4.14 (D5)
- net D6: now also U4.4 (D1); no longer U4.6 (D2)
- net D7: now also U4.13 (D4), U5.6; no longer U4.4 (D1)
- net GND: now also Y2.3, J4.1 (Pin_1); no longer R3.1
- net IRQ: no longer U5.4
- net RTC_CE: now also U4.15 (Q5); no longer U4.2 (Q0)
- net VCC: now also R3.1, J4.5 (Pin_5), JP2.3 (B); no longer U5.5
- net ~{RTC_RD}: now also JP2.1 (A); no longer U5.10
- net OUT_D0: now reaches U4.10 (Q3)
- net OUT_D0: now also J4.3 (Pin_3)
- net RTC_DOUT: now reaches U4.12 (Q4)
- net RTC_DOUT: now also U5.12
- net RTC_CLK renamed OUT_D2
- net OUT_D2: now also J4.4 (Pin_4); no longer U2.7 (SCLK)
- net RTC_IN renamed RTC_SCLK
- net RTC_SCLK: now also U2.7 (SCLK); no longer U5.12
- net RTC_WE renamed ~{RTC_WE}
- net ~{RTC_WE}: now also U4.2 (Q0); no longer U4.15 (Q5)
- net ~{INT}: no longer names the net of J3.22 (Pin_22)
- net ~{IRQ1}: no longer names the net of J3.37 (Pin_37)
- net ~{IRQ2}: no longer names the net of J3.77 (Pin_77)
- net ~{IRQ} renamed IN_D7
- net IN_D7: now also U5.5, J4.2 (Pin_2); no longer U5.6
- net ~{NMI}: no longer names the net of J3.66 (Pin_66)
- net ~{RFSH}: no longer names the net of J3.59 (Pin_59)
- new net ~{RTC_RD_ENA}: JP2.2 (C), U5.10, U5.4
- no-connect marks 53 -> 56
Other:
- title: Flock: RCBus FDC and RTC Module -> Flock: RCBUS FDC and RTC Module
- moved on the sheet: BT1, C7, J2, J3, JP1, R1, R3, U2, U5B, U5C, U5D, U5E
